Commit message: feat(webui): 3D 可视化 + LED 补发 + 主从跟随平滑限速版
机械臂可视化：
- 新增 arm.py（双臂配置 leader/follower + URDF 骨架解析，config/*.json）
- 页面 3D 视图（TF 树 + mesh 渲染）、关节轴显示开关、鼠标拖动交互
- 滑块 / 平滑到位 / 立即到位 / 回 home，实时关节角轮询

LED 状态修复：
- 位置指令 0x09 的 d[5] 高三位与 LED 颜色位同域，固件执行运动会顺带清灯
- WebConsole 记录 _led_state，goto / 整臂运动 / 跟随下发后按表补发灯色

主从跟随（平滑限速版，防过载报警）：
- 采样 / 控制双线程解耦：主动臂低频采样（默认 200 ms，5 Hz），
  从动臂高频插值控制（默认 20 ms，50 Hz）
- 梯形速度规划：斜坡起步（ramp_ms）→ 限速匀速（max_dps）→ 距离减速收尾，
  起步锚点为从动臂当前实际位置（capture），消除跳变冲击电流
- 死区吸收主动臂读数抖动；收敛后停发；旧参数 interval_ms 保留兼容
- 页面跟随栏新增采样/控制/限速/起步四个参数，徽标实时显示双频率与运动状态

测试：266 → 270 项（映射/限速/斜坡/起步锚点/参数记录/LED 补发等），全量通过

File: urdf/Romanbo.urdf (robot description, URDF)
Before this commit: robot Romanbo, 7 links, 6 joints
Joints:
- joint Romanbo_elbow_flex: axis 0 0 1 -> 0 0 -1; origin xyz=0.07960794 0.08406103 -0.0002 rpy=3.14159265 0 3.14159265 -> xyz=0.07960794 0.08406103 -0.0002 rpy=3.14159265 0 2.65159265
- joint Romanbo_gripper: limit lower=-0.95993 upper=0.95993 effort=10 velocity=10 -> lower=-0.33993 upper=1.57993 effort=10 velocity=10; origin xyz=0.00423498 0.01954648 0.04158296 rpy=1.57079633 0.00391439 -1.78416044 -> xyz=0.00423498 0.01954648 0.04158296 rpy=1.57079633 0.62391439 -1.78416044
- joint Romanbo_shoulder_lift: origin xyz=-0.02971501 -0.00649727 -0.0724 rpy=-1.57079633 0 0.21526495 -> xyz=-0.02971501 -0.00649727 -0.0724 rpy=-1.57079633 0.98 0.21526495
- joint Romanbo_shoulder_pan: origin xyz=0.04507171 0.00001297 0.04522959 rpy=3.14159265 0 3.14159265 -> xyz=0.04507171 0.00001297 0.04522959 rpy=3.14159265 0 -2.94159266
- joint Romanbo_wrist_flex: origin xyz=0.11429786 0.07147737 -0.0002 rpy=3.14159265 0 3.14159265 -> xyz=0.11429786 0.07147737 -0.0002 rpy=3.14159265 0 2.44159265
- joint Romanbo_wrist_roll: axis 0 0 1 -> 0 0 -1; origin xyz=-0.01404151 0.03907096 0.0003 rpy=1.57079633 -0.20262092 -2.79217493 -> xyz=-0.01404151 0.03907096 0.0003 rpy=-1.57079634 -1.28897173 0.34941774
